File: breadboard-psu.kicad_sch (KiCad schematic)
At the start: 11 parts, among them J1 USBC, U1 CH224K, U2 LM7805_TO220, U3 AMS1117-3.3

Commit message: upload
Parts:
- added J2: 5V_Rail, Connector_PinHeader_2.54mm:PinHeader_1x02_P2.54mm_Vertical, symbol Connector:Conn_01x02_Pin
- added J3: 3.3V_Rail, Connector_PinHeader_2.54mm:PinHeader_1x02_P2.54mm_Vertical, symbol Connector:Conn_01x02_Pin
- C1, C2, C3, C4: footprint Package_TO_SOT_THT:TO-220-3_Vertical -> Capacitor_SMD:C_0603_1608Metric
- D1: footprint (none) -> LED_SMD:LED_0603_1608Metric
- J1: footprint Package_DFN_QFN:Texas_RNQ0040A_WQFN-40-1EP_6x4mm_P0.4mm_EP4.7x2.7mm -> Connector_USB:USB_C_Receptacle_HRO_TYPE-C-31-M-12
- R1, R2: footprint Package_SO:SSOP-10-1EP_3.9x4.9mm_P1mm_EP2.1x3.3mm -> Resistor_SMD:R_0603_1608Metric
Connections:
- net +3.3V: now also R2.2, J3.1 (Pin_1)
- net +5V: now also J2.1 (Pin_1)
- net GND: now also J2.2 (Pin_2), J3.2 (Pin_2)
- net at R2.1: now also D1.2 (A); no longer U1.1 (VDD)
Other:
- moved on the sheet: R2
