File: breadboard-psu.kicad_pcb (KiCad board)
At the start: 4 copper layers, 20 x 20 mm, 13 parts, among them J1 USBC, J2 5V_Rail, J3 3.3V_Rail, U1 CH224K, U2 LM7805_TO220, U3 AMS1117-3.3

Commit message: finish up pcb
Parts:
- moved R2 66.3 mm to (168.0, 43.0)
- moved C4 62.9 mm to (165.0, 40.5), turned to 180 degrees
- moved C1 60.0 mm to (163.0, 42.5)
- moved C3 60.0 mm to (162.0, 38.0)
- moved R1 58.1 mm to (160.0, 42.5)
- moved C2 51.0 mm to (154.0, 46.0), turned to -90 degrees
- moved U3 1.80 mm to (165.0, 33.5), turned to 0 degrees
Routing:
- net GND: track 0.00 -> 36.6 mm, vias 5 -> 9
- net +3.3V: track 0.00 -> 23.2 mm
- net Net-(D1-K): track 0.00 -> 18.6 mm, vias 0 -> 2
- net +5V: track 6.26 -> 17.6 mm, vias 0 -> 1
- net Net-(U1-CFG1): track 0.00 -> 7.73 mm, vias 0 -> 2
- net +12V: track 3.54 -> 6.17 mm
- net Net-(D1-A): track 0.00 -> 2.52 mm
